File: BLDC driver.kicad_sch (KiCad schematic)
At the start: 0 parts

Commit message: removed excess files
Parts:
- added C1, C2, C3, C6: 470n, Capacitor_SMD:C_0603_1608Metric_Pad1.08x0.95mm_HandSolder, symbol Device:C_Small
- added C4: 100n, Capacitor_SMD:C_0603_1608Metric_Pad1.08x0.95mm_HandSolder, symbol Device:C
- added C5: 470u, Capacitor_THT:CP_Radial_D10.0mm_P7.50mm, symbol Device:C_Polarized
- added D1, D2, D3, D4, D5, D6: 1N5819, Diode_SMD:D_0603_1608Metric_Pad1.05x0.95mm_HandSolder, symbol Device:D_Schottky_Small
- added J1: Screw_Terminal_01x02, TerminalBlock:TerminalBlock_Altech_AK300-2_P5.00mm, symbol Connector:Screw_Terminal_01x02
- added J2: Screw_Terminal_01x03, TerminalBlock:TerminalBlock_Altech_AK300-3_P5.00mm, symbol Connector:Screw_Terminal_01x03
- added J3: Conn_02x06_Counter_Clockwise, Connector_PinHeader_2.54mm:PinHeader_2x06_P2.54mm_Vertical, symbol Connector_Generic:Conn_02x06_Counter_Clockwise
- added J4: Izlaz ocitavanje struje, Connector_PinHeader_2.54mm:PinHeader_1x04_P2.54mm_Vertical, symbol Connector:Conn_01x04_Pin
- added Q1, Q2, Q3, Q4, Q5, Q6: N0436N, Package_TO_SOT_SMD:TO-252-2, symbol Simulation_SPICE:NMOS
- added R1, R2, R3: 0.01, Resistor_SMD:R_Shunt_Vishay_WSR2_WSR3_KelvinConnection, symbol Device:R_US
- added R10, R11, R12, R13, R14, R9: 1k, Resistor_SMD:R_0603_1608Metric_Pad0.98x0.95mm_HandSolder, symbol Device:R_US
- added R15, R16, R17: 33k, Resistor_SMD:R_0603_1608Metric_Pad0.98x0.95mm_HandSolder, symbol Device:R_US
- added R18, R4, R5, R6, R7, R8: 20, Resistor_SMD:R_0603_1608Metric_Pad0.98x0.95mm_HandSolder, symbol Device:R_US
- added U1: MCP8027T-H/Y4X, Package_QFP:TQFP-48-1EP_7x7mm_P0.5mm_EP3.5x3.5mm, symbol 2026-06-16_11-31-29:MCP8027T-H_Y4X
Connections:
- new net: C3.2, J2.1 (Pin_1), Q1.3 (S), Q4.1 (D), U1.30 (PHA)
- new net: C1.2, J2.2 (Pin_2), Q2.3 (S), Q5.1 (D), U1.29 (PHB)
- new net: C2.2, J2.3 (Pin_3), Q3.3 (S), Q6.1 (D), U1.28 (PHC)
- new net: Q6.3 (S), R12.2, R3.1
- new net: Q3.2 (G), R6.2
- new net: R13.1, R16.2, U1.10 (ISENSE3-)
- new net: C2.1, D3.1 (K), D4.1 (K), U1.31 (VBC)
- new net: R10.1, R15.1, U1.13 (ISENSE2-)
- new net: R4.1, U1.27 (HSA)
- new net: Q1.2 (G), R4.2
- new net: C3.1, D1.1 (K), D6.1 (K), U1.33 (VBA)
- new net: C1.1, D2.1 (K), D5.1 (K), U1.32 (VBB)
- new net: C4.1, U1.42 (CAP2)
- new net: C4.2, U1.43 (CAP1)
- new net: R11.1, U1.11 (ISENSE3+)
- new net: R9.1, U1.14 (ISENSE2+)
- new net: R14.1, R17.2, U1.17 (I_SENSE1-)
- new net: R12.1, U1.18 (I_SENSE1+)
- new net: R7.1, U1.21 (LSA)
- new net: R8.1, U1.22 (LSB)
- new net: R18.1, U1.23 (LSC)
- new net: R6.1, U1.25 (HSC)
- new net: R5.1, U1.26 (HSB)
- new net: Q5.2 (G), R8.2
- new net: Q5.3 (S), R2.1, R9.2
- new net: Q4.2 (G), R7.2
- new net: Q4.3 (S), R1.1, R11.2
- new net: Q2.2 (G), R5.2
- new net: Q6.2 (G), R18.2
- new net 3V3: J3.7 (Pin_7), U1.40 (FB)
- new net D1: J3.8 (Pin_8), U1.3 (CE)
- new net D2: J3.9 (Pin_9), U1.15 (*ILIMIT_OUT)
- new net DE2: J3.10 (Pin_10), U1.44 (DE2)
- new net GND: C5.2, C6.1, D4.2 (A), D5.2 (A), D6.2 (A), J1.2 (Pin_2), J3.11 (Pin_11), J4.1 (Pin_1), R1.2, R10.2, R13.2, R14.2, R2.2, R3.2, U1.19 (PGND), U1.20 (PGND), U1.24 (PGND), U1.35 (PGND), U1.36 (PGND), U1.49 (PGND), U1.7 (PGND)
- new net I_OUT1: J4.4 (Pin_4), R17.1, U1.16 (I_OUT1)
- new net I_OUT2: J4.3 (Pin_3), R15.2, U1.12 (IOUT2)
- new net I_OUT3: J4.2 (Pin_2), R16.1, U1.9 (IOUT3)
- new net PWM1H: J3.6 (Pin_6), U1.2 (PWM1H)
- new net PWM1L: J3.5 (Pin_5), U1.1 (PWM1L)
- new net PWM2H: J3.4 (Pin_4), U1.48 (PWM2H)
- new net PWM2L: J3.3 (Pin_3), U1.47 (PWM2L)
- new net PWM3H: J3.2 (Pin_2), U1.46 (PWM3H)
- new net PWM3L: J3.1 (Pin_1), U1.45 (PWM3L)
- new net VCC: C5.1, C6.2, D1.2 (A), D2.2 (A), D3.2 (A), J1.1 (Pin_1), Q1.1 (D), Q2.1 (D), Q3.1 (D), U1.38 (VDD), U1.39 (VDD)
